File: KICAD8/COMMIT_5/H.A.V.O.C. PCB V 1.0.kicad_sch (KiCad schematic)
At the start: 75 parts, among them IC2 STM32H755IIT6, J10 Conn_02x10_Top_Bottom, J3 XT60-M, J5 Conn_Coaxial, J6 Conn_Coaxial, J7 Conn_02x10_Top_Bottom, M1 SERVO1, M2 SERVO2, M3 SERVO3, M4 SERVO4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

Commit message: In-progress Changes
HVT 1 -> 2, switching to a different format without pyro system. In between development, issues with HVT 1 from manufacturer, one from my design.
Parts:
- removed C50: 2.2uF, Capacitor_SMD:C_0805_2012Metric, symbol Device:C
- added 3v1: 3v3, TestPoint:TestPoint_Pad_1.5x1.5mm, symbol Connector:TestPoint
- added 5v1: 5V, TestPoint:TestPoint_Pad_1.5x1.5mm, symbol Connector:TestPoint
- added BOOT0, NRST1: OS102011MS2QN1, OS102011MS2QN1:SW_OS102011MS2QN1, symbol OS102011MS2QN1:OS102011MS2QN1
- added C23: 100nF, Capacitor_SMD:C_0805_2012Metric_Pad1.18x1.45mm_HandSolder, symbol Device:C
- added C53: 2.2 uF, Capacitor_SMD:C_0805_2012Metric_Pad1.18x1.45mm_HandSolder, symbol Device:C_Small
- added D4: YELLOW, LED_SMD:LED_0805_2012Metric_Pad1.15x1.40mm_HandSolder, symbol cr-2032:LED
- added NRST2: NRST, TestPoint:TestPoint_Pad_1.5x1.5mm, symbol Connector:TestPoint
- added R12, R14: 10k, Resistor_SMD:R_0805_2012Metric_Pad1.20x1.40mm_HandSolder, symbol Device:R
- added R13: 100, Resistor_SMD:R_0805_2012Metric_Pad1.20x1.40mm_HandSolder, symbol Device:R
- added S1: SERVO1, TestPoint:TestPoint_Pad_1.5x1.5mm, symbol Connector:TestPoint
- added S2: SERVO2, TestPoint:TestPoint_Pad_1.5x1.5mm, symbol Connector:TestPoint
- added S3: SERVO3, TestPoint:TestPoint_Pad_1.5x1.5mm, symbol Connector:TestPoint
- added S4: SERVO4, TestPoint:TestPoint_Pad_1.5x1.5mm, symbol Connector:TestPoint
- added S5: SERVO5, TestPoint:TestPoint_Pad_1.5x1.5mm, symbol Connector:TestPoint
- added SWCLK1: SWCLK, TestPoint:TestPoint_Pad_1.5x1.5mm, symbol Connector:TestPoint
- added Vbatbkp1: Vbckp, TestPoint:TestPoint_Pad_1.5x1.5mm, symbol Connector:TestPoint
- C1, C16, C17, C18, C2, C22: footprint Capacitor_SMD:C_0603_1608Metric -> Capacitor_SMD:C_0805_2012Metric_Pad1.18x1.45mm_HandSolder
- C19, C20, C21, C3, C30, C32, C4, C48: footprint Capacitor_SMD:C_0805_2012Metric -> Capacitor_SMD:C_0805_2012Metric_Pad1.18x1.45mm_HandSolder
- C33, C34, C35, C36, C37, C38, C39, C40, C41, C42, C43, C44, C45, C46, C47, C49: footprint Capacitor_SMD:C_0201_0603Metric -> Capacitor_SMD:C_0805_2012Metric_Pad1.18x1.45mm_HandSolder
- D16, D17, D6, D7: footprint LED_SMD:LED_0805_2012Metric -> LED_SMD:LED_0805_2012Metric_Pad1.15x1.40mm_HandSolder
- FB1: footprint Inductor_SMD:L_0402_1005Metric -> Inductor_SMD:L_0805_2012Metric_Pad1.05x1.20mm_HandSolder
- R10, R11, R15, R28, R29, R5, R6, R7, R8, R9: footprint Resistor_SMD:R_0805_2012Metric -> Resistor_SMD:R_0805_2012Metric_Pad1.20x1.40mm_HandSolder
- R16, R17, R18, R19, R20: footprint Resistor_SMD:R_0603_1608Metric -> Resistor_SMD:R_0805_2012Metric_Pad1.20x1.40mm_HandSolder
Connections:
- net +3V3: now also 3v1.1, BOOT0.1, NRST1.1
- net +5V: now also 5v1.1
- net BOOT0: now also BOOT0.2, D4.2 (A), R12.1, R12.2
- net GND: now also BOOT0.3, C23.2, C53.1, NRST1.3, R13.2
- net NRST: now also C23.1, NRST1.2, NRST2.1, R14.1, R14.2
- net SERVO1: now also S1.1
- net SERVO2: now also S2.1
- net SERVO3: now also S3.1
- net SERVO4: now also S4.1
- net SERVO5: now also S5.1
- net SWCLK: now also SWCLK1.1
- net VBat-backup: now also Vbatbkp1.1
- net at IC2.172 (VCAP_3): now also C53.2
- net AUX1_CONT: no longer names the net of IC2.150 (PD7)
- net AUX1_SIGNAL: no longer names the net of IC2.36 (PC2_C)
- net AUX2_CONT: no longer names the net of IC2.154 (PG10)
- net AUX2_SIGNAL: no longer names the net of IC2.37 (PC3_C)
- net DROGUE_CONT: no longer names the net of IC2.146 (PD3)
- net DROGUE_SIGNAL: no longer names the net of IC2.35 (PC1)
- net MAIN_CONT: no longer names the net of IC2.148 (PD5)
- net MAIN_SIGNAL: no longer names the net of IC2.34 (PC0)
- net PYRO_AUX1_FIRED: no longer names the net of IC2.149 (PD6)
- net PYRO_AUX2_FIRED: no longer names the net of IC2.153 (PG9)
- net PYRO_DROGUE_FIRED: no longer names the net of IC2.145 (PD2)
- net PYRO_MAIN_FIRED: no longer names the net of IC2.147 (PD4)
- new net: D4.1 (K), R13.1
- no-connect marks 57 -> 69
Other:
- removed sheet PYRO---TERMINALS
- sheet Power ports: added USB_D+, USB_D-; removed none
- note added: "BOOT-SWITCH"
- note added: "NRST-SWITCH"
- note added: "Revision Description HVT1: rev1 -> rev2: Made expansion connectors symmetric for power/gnd HVT1: rev2 -> rev3: Removed 2 IO Expansion slots due to PCB Size limitations HVT2: rev0 -> rev1: Removed pyro capability"
- note added: "Test Points"
- note removed: "Revision Description rev1 -> rev2: Made expansion connectors symmetric for power/gnd rev2 -> rev3: Removed 2 IO Expansion slots due to PCB Size limitations"
- moved on the sheet: BZ1, C16, C17, C18, C19, C30, C32, C33, C34, C35, C36, C37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

Commit message: Intermediary Progress on HVT2
Removed pyro circuits for cost reasons, most of layout completed, traces need to be routed still
Connections:
- net VBAT_SWITCH is gone; now on net VBAT: R28.2
Other:
- sheet Power ports: added none; removed 3v3-out, 5v-out, 5v-out-usb, GND, USB_D+, USB_D-, VBAT_SWITCH
